File: IDHolder_Cover.brd (EAGLE design)
At the start: 64 x 99.5 mm, 24 parts

Commit message: Laid out traces
Parts:
- removed E$10: (no value), CougsInSpace-Aesthetics:SIGN-BRADLEY
- removed E$14: (no value), led:LZ4-40U600
- removed E$17: (no value), CougsInSpace-DiscreteSemi:UDFN-6
- removed E$18: (no value), CougsInSpace-Clocks:SMD-3225
- removed E$21: (no value), CougsInSpace-Connectors:U.FL
- removed E$23: (no value), CougsInSpace-IC-Power:QFN-TPS61089
- removed E$25, E$26, E$27, E$29, E$30, E$31: (no value), CougsInSpace-LEDs:1608-POL
- added DS1: (no value), led:LZ4-40U600
- added DS2, DS3, DS4, DS5, DS6, DS7: (no value), CougsInSpace-LEDs:1608-POL
- added R5: (no value), CougsInSpace-Capacitors:1608
- added U3: (no value), analog-devices:BGA_CB11
- added U4: (no value), CougsInSpace-IC-Power:QFN-TPS61089
- added U5: (no value), CougsInSpace-DiscreteSemi:UDFN-6
- added Y1: (no value), CougsInSpace-Clocks:SMD-3225
- E$1: device analog-devices:BGA_CB11 -> CougsInSpace-Aesthetics:SIGN-BRADLEY
- moved E$1 81.5 mm to (-28.6, -28.9), turned to 0 degrees
- renumbered E$2 to U2, E$22 to Z1, E$24 to U6, E$28 to U1, E$3 to R3, E$4 to R4, E$5 to J1, E$6 to C2, E$7 to C1, E$8 to R1, E$9 to R2
Connections:
- new net ANT_N: R5.1, U3.C1
- new net ANT_P: R5.2, U3.B1
- new net S$3: U2.25, U2.26
- net D_0: now also U3.D1; no longer E$1.D1
- net D_1: now also U3.D2; no longer E$1.D2
- net D_2: now also U3.D3; no longer E$1.D3
- net D_3: now also U3.C3; no longer E$1.C3
- net D_4: now also U3.B3; no longer E$1.B3
- net D_5: now also U3.A3; no longer E$1.A3
- net D_6: now also U3.A2; no longer E$1.A2
- net D_7: now also U3.A1; no longer E$1.A1
- net OUT: no longer E$21.CENTER
- net OUT_NEG: no longer E$21.SHIELD@1, E$21.SHIELD@13, E$21.SHIELD@2
- net S$20: now also DS2.A, DS3.A, DS4.A, DS5.A, DS6.A, DS7.A, U5.PAD-BTM, U5.PAD-TOP; no longer E$17.PAD-BTM, E$17.PAD-TOP, E$25.A, E$26.A, E$27.A, E$29.A, E$30.A, E$31.A
- net S$21: now also DS7.C, U5.4; no longer E$17.4, E$25.C
- net S$22: now also DS6.C, U5.5; no longer E$17.5, E$26.C
- net S$23: now also DS5.C, U5.6; no longer E$17.6, E$27.C
- net S$24: now also DS4.C, U5.1; no longer E$17.1, E$29.C
- net S$25: now also DS3.C, U5.2; no longer E$17.2, E$30.C
- net S$26: now also DS2.C, U5.3; no longer E$17.3, E$31.C
- net S$27: now also U2.16
- net S$31: now also Y1.1; no longer E$18.1
- net S$32: now also Y1.3; no longer E$18.3
- net S$34: now also Y1.2, Y1.4; no longer E$18.2, E$18.4
- net S$43: now also DS1.1, DS1.2, DS1.3, DS1.4, DS1.5, DS1.6, DS1.7, DS1.8; no longer E$14.1, E$14.2, E$14.3, E$14.4, E$14.5, E$14.6, E$14.7, E$14.8
- net S$44: now also DS1.TH; no longer E$14.TH
- net S$47: now also U4.11; no longer E$23.11
- net S$51: now also U4.10; no longer E$23.10
- net S$52: now also U4.2; no longer E$23.2
- net S$53: now also U4.1; no longer E$23.1
Routing:
- net S$27: track 0.00 -> 198.2 mm, vias 0 -> 6
- net S$61: track 0.00 -> 168.4 mm
- net S$53: track 0.00 -> 102.0 mm
- net ANT_N: track 0.00 -> 69.8 mm
- net ANT_P: track 0.00 -> 69.7 mm
- net OUT: track 26.1 -> 82.2 mm
- net S$47: track 0.00 -> 47.3 mm
- net S$3: track 0.00 -> 46.3 mm
- net OUT_NEG: track 35.7 -> 6.98 mm, vias 6 -> 5
- net S$26: track 0.00 -> 28.7 mm
- net S$20: track 0.00 -> 25.5 mm
- net S$25: track 0.00 -> 24.2 mm
- net S$43: track 0.00 -> 19.7 mm
- net S$24: track 0.00 -> 19.5 mm
- net S$23: track 0.00 -> 14.1 mm
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- added copper zone on layer 1, net 1
- added copper zone on layer 1, net 2
- added copper zone on layer 1, net 3
- added copper zone on layer 1, net ANT_N
- added copper zone on layer 1, net ANT_P
- added copper zone on layer 1, net S$43
- added copper zone on layer 1, net S$47
- added copper zone on layer 1, net S$53
- added copper zone on layer 1, net TRIANGLE
- added copper zone on layer 1, net TRIANGLE1
- added copper zone on layer 1, net TRIANGLE2

Commit message: Created center piece
Parts:
- added C3: (no value), CougsInSpace-Capacitors:1608
- moved E$1 1.70 mm to (-28.6, -30.6)
- moved U1 1.61 mm to (-15.0, 49.3)
- moved DS1 0.14 mm to (-20.1, 45.7)
Connections:
- net S$43 renamed S$4
- removed net S$27: U2.16, U2.32
- new net S$33: J1.22
- new net S$35: U6.A6
- new net S$36: U6.D2
- new net S$37: U6.D5
- new net S$38: R3.2
- new net S$39: U4.5, U4.6
- new net S$40: J1.1, J1.8
- new net S$41: C3.2, U6.J6
- new net S$42: C3.1, U6.H6
- new net S$5: U2.16
- new net S$6: U2.32
- net S$15: no longer U6.A6, U6.D5
- net S$16: no longer U6.D2
- net S$2: no longer R3.2
- net S$9: no longer J1.22
Routing:
- net S$61: track 168.4 -> 208.7 mm
- net ANT_N: track 69.8 -> 29.7 mm
- net ANT_P: track 69.7 -> 29.6 mm
- net S$40: track 0.00 -> 25.6 mm
- net S$5: track 0.00 -> 21.7 mm, vias 0 -> 1
- net S$39: track 0.00 -> 13.4 mm
- net S$27: track 198.2 -> 186.5 mm, vias 6 -> 2
- net S$10: track 0.00 -> 11.6 mm, vias 0 -> 2
- net S$15: track 20.1 -> 9.11 mm, vias 3 -> 1
- net S$9: track 13.5 -> 6.65 mm, vias 2 -> 1
- net S$2: track 7.81 -> 1.40 mm, vias 2 -> 1
- net S$4: track 19.7 -> 24.6 mm
- net S$16: track 15.9 -> 11.2 mm, vias 2 -> 1
- net S$42: track 0.00 -> 2.64 mm
- net S$44: track 13.2 -> 10.8 mm
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- added copper zone on layer 16, net BOTTOM
- removed copper zone on layer 1, net S$4
Other:
- outline, holes or cut-outs redrawn
